File: hardware/main_board.kicad_sch (KiCad schematic)
At the start: 67 parts, among them J1 Eurorack Power, J2 Conn_01x08, J3 Conn_01x08, J4 Conn_01x10, J6 Conn_01x10, Q1 2N3904, Q2 2N3904, Q3 2N3904, Q4 2N3904, U1 L7805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

Commit message: updated bom
Parts:
- R29: value 18K -> 18k
- R30: value 6.8K -> 6.8k
- R31: value 30K -> 30k
- R32: value 12K -> 12k
Changed lines of the file:
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@@
 			)
 		)
-		(property "Value" "6.8K"
+		(property "Value" "6.8k"
 			(at 107.696 152.654 90)
 			(effects
@@
 			)
 		)
-		(property "Value" "30K"
+		(property "Value" "30k"
 			(at 127 140.97 90)
 			(effects
@@
 			)
 		)
-		(property "Value" "18K"
+		(property "Value" "18k"
 			(at 107.95 140.97 90)
 			(effects
@@
 			)
 		)
-		(property "Value" "12K"
+		(property "Value" "12k"
 			(at 126.746 152.654 90)
 			(effects
