File: hardware/quadulator.kicad_pcb (KiCad board)
At the start: 2 copper layers, 144.1 x 181.4 mm, 128 parts, among them J1 Eurorack Power, J10 3.5mm jack, J11 3.5mm jack, J12 3.5mm jack, J13 3.5mm jack, J14 3.5mm jack, J15 3.5mm jack, J16 3.5mm jack, J17 3.5mm jack, J18 3.5mm jack, J19 3.5mm jack, J2 Conn_01x08, J20 3.5mm jack, J21 3.5mm jack, J3 Conn_01x08, J4 Conn_01x10, J5 Conn_01x08, J6 Conn_01x10, J7 Conn_01x08, J8 Conn_01x10, J9 Conn_01x10, Q1 2N3904, Q2 2N3904, Q3 2N3904, Q4 2N3904, SW1 SW_Push, SW2 SW_Push, SW3 SW_Push, SW4 SW_Push, SW5 SW_Push, U1 L7805, U2 Pico, U3 MCP6004, U4 CD4051B, U5 TL074, U6 74HC595, U7 TL074

Commit message: updated bom
Parts:
- R29: value 18K -> 18k
- R30: value 6.8K -> 6.8k
- R31: value 30K -> 30k
- R32: value 12K -> 12k
Changed lines of the file:
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@@
 			)
 		)
-		(property "Value" "18K"
+		(property "Value" "18k"
 			(at 3.81 2.37 90)
 			(layer "F.Fab")
@@
 			)
 		)
-		(property "Value" "30K"
+		(property "Value" "30k"
 			(at 3.81 2.37 90)
 			(layer "F.Fab")
@@
 			)
 		)
-		(property "Value" "6.8K"
+		(property "Value" "6.8k"
 			(at 3.81 2.37 0)
 			(layer "F.Fab")
@@
 			)
 		)
-		(property "Value" "12K"
+		(property "Value" "12k"
 			(at 3.81 2.37 0)
 			(layer "F.Fab")
